Commit message: minor improvements

File: stepper_motor_control/urdf/robot_controller/robot_controller.macro.xacro (robot description, xacro)
@@ -7,7 +7,4 @@
         *origin
         " >
-        <!-- Note : for now i'm using dark grey color for the motors as the mesh does not display the true colors of the motors (.stl is not made for this)
-         I left the .dae file which should display a better visual if you can make it work
-         I'm also spawning a different shaft on the motor which is only a display solution, the size is then not respected -->
     <material name="white">
         <color rgba="1 1 1 1"/>
@@ -35,8 +32,8 @@
         <visual>
             <geometry>
-                <mesh filename="file://$(find stepper_motor_control)/meshes/PD4-C6018L4204-E-08(1).dae" scale="0.01 0.01 0.01"/>
-            </geometry>
-            <!-- <material name="motor"> -->
-            <!-- </material> -->
+                <mesh filename="file://$(find stepper_motor_control)/meshes/PD4-C6018L4204-E-08.stl" scale="0.01 0.01 0.01"/>
+            </geometry>
+            <material name="motor">
+            </material>
         </visual>
         <collision>

File: stepper_motor_control/urdf/robot_controller/robot_controller.ros2_control.xacro (robot description, xacro)
@@ -10,5 +10,5 @@
         <ros2_control name="${name}" type="system"> <!-- the type can be different than system (actuator) ? and one control hardware for each motor ?? -->
             <hardware>
-                <plugin>canopen_ros2_control/Cia402System</plugin>
+                <plugin>canopen_ros2_control/RobotSystem</plugin>
                 <param name="bus_config">${bus_config}</param>
                 <param name="master_config">${master_config}</param>
@@ -25,5 +25,6 @@
             </joint> -->
             <joint name="${prefix}third_shaft_joint">
-                <param name="node_id">2</param>
+                <param name="device_name">third_shaft_joint</param>
+                <state_interface name="position" />
             </joint>
             <!-- <joint name="${prefix}fourth_shaft_joint">
