Commit message: Merged the two packages and minor launch changes

File: stepper_motor_control/urdf/robot_controller/robot_controller.ros2_control.xacro (robot description, xacro)
@@ -33,20 +33,4 @@
             </joint> -->
         </ros2_control>
-        <!-- The following plugin allows the compatibility with the controllers (see in the launch file), when running, calling the services won't make the motors move, you have to use the plugin's commands instead -->
-        <!-- <ros2_control name="${name}" type="system">
-            <hardware>
-                <plugin>canopen_ros2_control/Cia402System</plugin>
-                <param name="bus_config">${bus_config}</param>
-                <param name="master_config">${master_config}</param>
-                <param name="can_interface_name">${can_interface_name}</param>
-                <param name="master_bin">"${master_bin}"</param>
-            </hardware>
-            <joint name="${prefix}first_shaft_joint">
-                <param name="node_id">1</param>
-            </joint>
-            <joint name="${prefix}second_shaft_joint">
-                <param name="node_id">2</param>
-            </joint>
-        </ros2_control> -->
     </xacro:macro>
 </robot>

Commit message: Newy added features and securties for motors control

File: stepper_motor_control/urdf/robot_controller/robot_controller.ros2_control.xacro (robot description, xacro)
@@ -19,6 +19,6 @@
                 <param name="device_name">first_shaft_joint</param>
                 <state_interface name="position" />
-            </joint> -->
-            <!-- <joint name="${prefix}second_shaft_joint">
+            </joint>
+            <joint name="${prefix}second_shaft_joint">
                 <param name="device_name">second_shaft_joint</param>
                 <state_interface name="position" />
